Commit message: Update mesh file paths to use 'file://' syntax
Signed-off-by: Irene Bandera Moreno <ibanderam@gmail.com>

File: robotiq_description/urdf/robotiq_2f_140_macro.urdf.xacro (robot description, xacro)
@@ -54,5 +54,5 @@
           <origin xyz="0 0 0" rpy="0 0 0" />
           <geometry>
-            <mesh filename="package://robotiq_description/meshes/visual/2f_140/robotiq_2f_140_base_link.stl" />
+            <mesh filename="file://$(find robotiq_description)/meshes/visual/2f_140/robotiq_2f_140_base_link.stl" />
           </geometry>
           <material name="">
@@ -63,5 +63,5 @@
           <origin xyz="0 0 0" rpy="0 0 0" />
           <geometry>
-            <mesh filename="package://robotiq_description/meshes/collision/2f_140/robotiq_2f_140_base_link.stl" />
+            <mesh filename="file://$(find robotiq_description)/meshes/collision/2f_140/robotiq_2f_140_base_link.stl" />
           </geometry>
         </collision>
