Commit message: Change mimic joint type from revolut to continuous
Signed-off-by: Irene Bandera Moreno <ibanderam@gmail.com>

File: robotiq_description/urdf/robotiq_2f_140.xacro (robot description, xacro)
@@ -155,5 +155,5 @@
   </xacro:macro>
   <xacro:macro name="right_outer_knuckle_joint" params="prefix">
-    <joint name="${prefix}right_outer_knuckle_joint" type="revolute">
+    <joint name="${prefix}right_outer_knuckle_joint" type="continuous">
       <origin xyz="0 0.030601 0.054905" rpy="${pi / 2 + .725} 0 ${pi}" />
       <parent link="${prefix}robotiq_140_base_link" />
@@ -174,5 +174,5 @@
   </xacro:macro>
   <xacro:macro name="inner_knuckle_joint" params="prefix fingerprefix reflect">
-    <joint name="${prefix}${fingerprefix}_inner_knuckle_joint" type="revolute">
+    <joint name="${prefix}${fingerprefix}_inner_knuckle_joint" type="continuous">
       <origin xyz="0 ${reflect * -0.0127} 0.06142" rpy="${pi / 2 + .725} 0 ${(reflect - 1) * pi / 2}" />
       <parent link="${prefix}robotiq_140_base_link" />
@@ -184,5 +184,5 @@
   </xacro:macro>
   <xacro:macro name="inner_finger_joint" params="prefix fingerprefix">
-    <joint name="${prefix}${fingerprefix}_inner_finger_joint" type="revolute">
+    <joint name="${prefix}${fingerprefix}_inner_finger_joint" type="continuous">
       <origin xyz="0 0.0817554015893473 -0.0282203446692936" rpy="-0.725 0 0" />
       <parent link="${prefix}${fingerprefix}_outer_finger" />

Commit message: Align Robotiq 140 with Robotiq 85 updates (#1)
* Update mesh file paths to use 'file://' syntax

Signed-off-by: Irene Bandera Moreno <ibanderam@gmail.com>

* Change mimic joint type from revolut to continuous

Signed-off-by: Irene Bandera Moreno <ibanderam@gmail.com>

---------

Signed-off-by: Irene Bandera Moreno <ibanderam@gmail.com>

File: robotiq_description/urdf/robotiq_2f_140.xacro (robot description, xacro)
@@ -17,5 +17,5 @@
         <origin xyz="0 0 0" rpy="0 0 0" />
         <geometry>
-          <mesh filename="package://robotiq_description/meshes/visual/2f_140/robotiq_2f_${stroke}_outer_knuckle.stl" />
+          <mesh filename="file://$(find robotiq_description)/meshes/visual/2f_140/robotiq_2f_${stroke}_outer_knuckle.stl" />
         </geometry>
         <material name="">
@@ -26,5 +26,5 @@
         <origin xyz="0 0 0" rpy="0 0 0" />
         <geometry>
-          <mesh filename="package://robotiq_description/meshes/collision/2f_140/robotiq_2f_${stroke}_outer_knuckle.stl" />
+          <mesh filename="file://$(find robotiq_description)/meshes/collision/2f_140/robotiq_2f_${stroke}_outer_knuckle.stl" />
         </geometry>
       </collision>
@@ -47,5 +47,5 @@
         <origin xyz="0 0 0" rpy="0 0 0" />
         <geometry>
-          <mesh filename="package://robotiq_description/meshes/visual/2f_140/robotiq_2f_${stroke}_outer_finger.stl" />
+          <mesh filename="file://$(find robotiq_description)/meshes/visual/2f_140/robotiq_2f_${stroke}_outer_finger.stl" />
         </geometry>
         <material name="">
@@ -56,5 +56,5 @@
         <origin xyz="0 0 0" rpy="0 0 0" />
         <geometry>
-          <mesh filename="package://robotiq_description/meshes/collision/2f_140/robotiq_2f_${stroke}_outer_finger.stl" />
+          <mesh filename="file://$(find robotiq_description)/meshes/collision/2f_140/robotiq_2f_${stroke}_outer_finger.stl" />
         </geometry>
       </collision>
@@ -77,5 +77,5 @@
         <origin xyz="0 0 0" rpy="0 0 0" />
         <geometry>
-          <mesh filename="package://robotiq_description/meshes/visual/2f_140/robotiq_2f_${stroke}_inner_knuckle.stl" />
+          <mesh filename="file://$(find robotiq_description)/meshes/visual/2f_140/robotiq_2f_${stroke}_inner_knuckle.stl" />
         </geometry>
         <material name="">
@@ -86,5 +86,5 @@
         <origin xyz="0 0 0" rpy="0 0 0" />
         <geometry>
-          <mesh filename="package://robotiq_description/meshes/collision/2f_140/robotiq_2f_${stroke}_inner_knuckle.stl" />
+          <mesh filename="file://$(find robotiq_description)/meshes/collision/2f_140/robotiq_2f_${stroke}_inner_knuckle.stl" />
         </geometry>
       </collision>
@@ -107,5 +107,5 @@
         <origin xyz="0 0 0" rpy="0 0 0" />
         <geometry>
-          <mesh filename="package://robotiq_description/meshes/visual/2f_140/robotiq_2f_${stroke}_inner_finger.stl" />
+          <mesh filename="file://$(find robotiq_description)/meshes/visual/2f_140/robotiq_2f_${stroke}_inner_finger.stl" />
         </geometry>
         <material name="">
@@ -116,5 +116,5 @@
         <origin xyz="0 0 0" rpy="0 0 0" />
         <geometry>
-          <mesh filename="package://robotiq_description/meshes/collision/2f_140/robotiq_2f_${stroke}_inner_finger.stl" />
+          <mesh filename="file://$(find robotiq_description)/meshes/collision/2f_140/robotiq_2f_${stroke}_inner_finger.stl" />
         </geometry>
       </collision>
@@ -155,5 +155,5 @@
   </xacro:macro>
   <xacro:macro name="right_outer_knuckle_joint" params="prefix">
-    <joint name="${prefix}right_outer_knuckle_joint" type="revolute">
+    <joint name="${prefix}right_outer_knuckle_joint" type="continuous">
       <origin xyz="0 0.030601 0.054905" rpy="${pi / 2 + .725} 0 ${pi}" />
       <parent link="${prefix}robotiq_140_base_link" />
@@ -174,5 +174,5 @@
   </xacro:macro>
   <xacro:macro name="inner_knuckle_joint" params="prefix fingerprefix reflect">
-    <joint name="${prefix}${fingerprefix}_inner_knuckle_joint" type="revolute">
+    <joint name="${prefix}${fingerprefix}_inner_knuckle_joint" type="continuous">
       <origin xyz="0 ${reflect * -0.0127} 0.06142" rpy="${pi / 2 + .725} 0 ${(reflect - 1) * pi / 2}" />
       <parent link="${prefix}robotiq_140_base_link" />
@@ -184,5 +184,5 @@
   </xacro:macro>
   <xacro:macro name="inner_finger_joint" params="prefix fingerprefix">
-    <joint name="${prefix}${fingerprefix}_inner_finger_joint" type="revolute">
+    <joint name="${prefix}${fingerprefix}_inner_finger_joint" type="continuous">
       <origin xyz="0 0.0817554015893473 -0.0282203446692936" rpy="-0.725 0 0" />
       <parent link="${prefix}${fingerprefix}_outer_finger" />
